Commit message: added the ros2_control archi to repo

File: src/rover_arm_description/urdf/rover_arm_raw.xacro (robot description, xacro)
@@ -254,2 +254,4 @@
   </gazebo>
 </robot>
+<!-- This file should only start with the robot we will add separately the hardware and software plugins later
+So I don't want to spoil this file by adding plugins here-->

File: src/rover_arm_description/urdf/rover_arm_real.xacro (robot description, xacro)
@@ -230,6 +230,8 @@
     <hardware>
       <plugin>rover_arm_hardware/RoverArmHardware</plugin>
-      <param name="serial_port">/dev/ttyACM0</param>
-      <param name="baud_rate">115200</param>
+      <xacro:property name="serial_port" value="/dev/ttyACM0"/>
+      <xacro:property name="baud_rate" value="115200"/>
+      <param name="serial_port">${serial_port}</param>      <!--- If by any chance the port changes we can edit here-->
+      <param name="baud_rate">${baud_rate}</param>
     </hardware>
     <xacro:joint_interface joint_name="base_link_joint" />

File: src/rover_arm_description/urdf/rover_arm_sim.xacro (robot description, xacro)
@@ -204,5 +204,5 @@
   <xacro:blue_pla link_name="camera_mount_link"/>
   <link name="gripper_camera_optical_frame"/>
-  <link name="zed_camera_optical_frame"/>
+ <!--  <link name="zed_camera_optical_frame"/>   Commented for now, uncomment after properly establishing joint-->
   <joint name="stand_link_joint" type="fixed">
     <origin xyz="0.0 0.0 0.0" rpy="0.0 0.0 0.0" />
