Commit message: Updated

File: src/rover_arm_description/urdf/rover_arm_real.xacro (robot description, xacro)
@@ -230,8 +230,7 @@
     <hardware>
       <plugin>rover_arm_hardware/RoverArmHardware</plugin>
-      <xacro:property name="serial_port" value="/dev/ttyACM0"/>
-      <xacro:property name="baud_rate" value="115200"/>
-      <param name="serial_port">${serial_port}</param>      <!--- If by any chance the port changes we can edit here-->
-      <param name="baud_rate">${baud_rate}</param>
+      <param name="kp">40.0</param>
+      <param name="ki">5.0</param>
+      <param name="pwm_limit">255.0</param>
     </hardware>
     <xacro:joint_interface joint_name="base_link_joint" />
